File: dds-function-gen2.kicad_pcb (KiCad board)
At the start: 2 copper layers, 85.1 x 58.4 mm, 32 parts, among them IC1 ATMEGA168A-A, U1 LM317EMP, U2 LM337T, U3 LM317EMP, U5 AD9833, X1 20Mhz

Commit message: PCB's in progress
Parts:
- moved DS1 60.7 mm to (252.6, 96.4)
- moved U5 56.1 mm to (232.5, 110.4), turned to 90 degrees
- moved IC1 48.5 mm to (224.9, 98.2)
- moved X1 37.1 mm to (212.9, 119.1)
- moved C7 36.5 mm to (211.7, 123.5)
- moved C6 32.4 mm to (210.0, 119.8)
- moved C5 31.7 mm to (208.0, 119.7)
- moved C8 31.6 mm to (205.8, 119.6)
- moved R6 29.4 mm to (206.9, 113.1), turned to 270 degrees
- moved C10 29.0 mm to (203.9, 92.5)
- moved C2 27.7 mm to (197.4, 120.3)
- moved C1 27.4 mm to (197.9, 117.1)
- moved C9 25.4 mm to (197.1, 112.1)
- moved D6 25.4 mm to (202.0, 111.3)
- moved R4 24.4 mm to (202.9, 104.8)
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Routing:
- net AGND: track 9.00 -> 0.00 mm
- net (no net): track 0.00 -> 9.00 mm
