File: dds-function-gen2.sch (KiCad schematic (older format))
At the start: 32 parts, among them IC1 ATMEGA168A-A, U1 LM317EMP, U2 LM337T, U3 LM317EMP, U5 AD9833, X1 20Mhz

Commit message: PCB's in progress
Other:
- note added: "0.1a"
- note added: "DDS David Mebane (Digikutz)9@gmail.com"
Changed lines of the file:
@@
 Sheet 1 1
 Title ""
-Date "19 feb 2014"
+Date "12 mar 2014"
 Rev ""
 Comp ""
@@
 Wire Wire Line
 	2200 3750 1950 3750
+Text Notes 7350 7550 0    60   ~ 0
+DDS                  David Mebane (Digikutz)9@gmail.com
+Text Notes 10700 7650 0    60   ~ 0
+0.1a
 $EndSCHEMATC
